File: KiCAD/EMS-Cast/EMS-Cast.kicad_sch (KiCad schematic)
At the start: 42 parts, among them IC1 LH1546ADF, IC2 LH1546ADF, IC3 LH1546ADF, IC4 LH1546ADF, J1 1720430202, J2 5-103166-1, J3 5-103166-1, Q1 STD25NF20, Q2 STD25NF20, Q3 STD25NF20, Q4 STD25NF20, SW2 SW_Push, SW3 SW_Push, U1 AD5252BRUZ10-RL7, U2 VOM1271T, U3 VOM1271T, U4 KF80BDT

Commit message: Multiple Changes
- Updated KICAD for proposal images
- Added Arduino code folder with basic .ino code (basic requirement and temporary pin mappings)
Parts:
- removed U4: KF80BDT, Package_TO_SOT_SMD:TO-252-2, symbol Regulator_Linear:KF80BDT
- added BT1: Battery_Cell, footprints:BatteryHolder_Keystone_106_1x20mm, symbol HPS:Battery_Cell
- added C11, C12, C13, C16: C_0805_0.1uf, footprints:C_0805_2012Metric, symbol HPS:C_0805_0.1uf
- added C14, C15: 22p, footprints:C_0805_2012Metric, symbol HPS:C_0805_22pf
- added C17, C20: C_Polarized, symbol Device:C_Polarized
- added C18: .01u, Capacitor_SMD:CP_Elec_6.3x3, symbol Device:C
- added D1: LED_0805, footprints:LED_0805_2012Metric, symbol HPS:LED_0805
- added D5: 1N5820, Diode_THT:D_DO-201AD_P15.24mm_Horizontal, symbol Diode:1N5820
- added IC5: KF33BDT-TR, EMS_lib:TO228P972X240-3N, symbol EMS_lib:KF33BDT-TR
- added J4: ~, EMS_lib:FFC_I2C_General, symbol EMS_lib:FFC_I2C_General
- added J5: Conn_01x06, footprints:PinHeader_1x06_P2.54mm_Vertical, symbol HPS:Conn_01x06
- added J7: Conn_02x03_Odd_Even, footprints:PinHeader_2x03_P2.54mm_Vertical, symbol HPS:Conn_02x03_Odd_Even
- added L1: 68u, symbol Device:L
- added PS1: IA0503D, Converter_DCDC:Converter_DCDC_XP_POWER-IAxxxxD_THT, symbol Converter_DCDC:IA0503D
- added R13, R14: 1K, Resistor_SMD:R_0805_2012Metric, symbol Device:R
- added R17: 10KΩ, footprints:R_0805_2012Metric, symbol HPS:R_0805_10K
- added R18: R_0805_2.2K, footprints:R_0805_2012Metric, symbol HPS:R_0805_2.2K
- added RX_TP1, TX_TP1, VBAT_TP1: TestPoint, footprints:TestPoint_THTPad_D2.0mm_Drill1.0mm, symbol HPS:TestPoint
- added SW1: Omron_B3F_SPST, footprints:SW_SPST_Omron_B3FS-100xP, symbol HPS:Omron_B3F_SPST
- added U4: ATmega328-PU, footprints:DIP-28_W7.62mm, symbol HPS:ATmega328-PU
- added U5: DS1307_DIP-8, footprints:DIP-8_W7.62mm, symbol HPS:DS1307_DIP-8
- added U6: XL1509-5.0, Package_SO:SOIC-8_3.9x4.9mm_P1.27mm, symbol Regulator_Switching:XL1509-5.0
- added U7: 74AUC1G79, symbol 74xGxx:74AUC1G79
- added Y1: Crystal 16MHZ, footprints:Crystal_SMD_HC49-SD, symbol HPS:Crystal_16MHz
- added Y2: Crystal_32768Hz, footprints:Crystal_SMD_2Pin_3.2x1.5mm, symbol HPS:Crystal_32768Hz
- C1: value .01u -> 1u; footprint Capacitor_THT:C_Axial_L17.0mm_D6.5mm_P25.00mm_Horizontal -> Capacitor_SMD:CP_Elec_6.3x3
- C10, C3, C4, C5, C6, C7, C8, C9: footprint Capacitor_THT:C_Axial_L17.0mm_D6.5mm_P25.00mm_Horizontal -> EMS_lib:K104K15X7RF53H5
- C2: footprint Capacitor_THT:C_Axial_L17.0mm_D6.5mm_P25.00mm_Horizontal -> Capacitor_SMD:CP_Elec_6.3x3
- D2, D3: footprint LED_THT:LED_D8.0mm -> EMS_lib:WL-TMRC_3MM
- R1, R11, R12, R2, R3, R4, R5, R6, R7, R8: footprint Resistor_THT:R_Axial_DIN0204_L3.6mm_D1.6mm_P1.90mm_Vertical -> Resistor_SMD:R_0805_2012Metric
- R10: value 1K -> 4.7k; footprint Resistor_THT:R_Axial_DIN0204_L3.6mm_D1.6mm_P1.90mm_Vertical -> Resistor_SMD:R_0805_2012Metric
- R9: value 1K -> 4.7K; footprint Resistor_THT:R_Axial_DIN0204_L3.6mm_D1.6mm_P1.90mm_Vertical -> Resistor_SMD:R_0805_2012Metric
Connections:
- net +3.3V: now also R10.2, R9.2, J4.1 (Vdd), R17.2
- net CH1_EN_1: now also U4.6 (PD4); no longer A1.7 (D4)
- net CH1_EN_2: now also U4.11 (OC0B/PD5); no longer A1.8 (D5)
- net CH2_EN_1: now also U4.12 (OC0A/PD6); no longer A1.9 (D6)
- net CH2_EN_2: now also U4.13 (PD7); no longer A1.10 (D7)
- net GND: now also BT1.2 (-), C11.2, C12.2, C13.2, C14.2, C15.2, D1.1 (K), IC5.4 (GND_TAB), J4.4 (GND), J5.1 (Pin_1), J5.2 (Pin_2), J7.6 (Pin_6), SW1.3 (B), SW1.4 (B), U4.22 (GND), U4.8 (GND), U5.4 (GND)
- net SCLK: now also R10.1, J4.3 (SCL), U4.28 (SCL/PC5); no longer A1.24 (A5)
- net SDA: now also R9.1, J4.2 (SDA), U4.27 (SDA/PC4); no longer A1.23 (A4)
- net SW_CH1: now also U4.14 (PB0); no longer A1.11 (D8)
- net SW_CH2: now also U4.15 (OC1A/PB1); no longer A1.12 (D9)
- net at D2.2 (A): now also R13.1; no longer R9.1
- net at A1.22 (A3): no longer R9.2
- net at D3.2 (A): now also R14.1; no longer R10.1
- net at A1.21 (A2): no longer R10.2
- net VCC: now reaches A1.30 (VIN), C2.1
- net VCC: now also C13.1, IC5.3 (OUTPUT), J7.2 (Pin_2), U4.20 (AVCC), U4.7 (VCC), U5.8 (VCC)
- net at C1.1, J1.1: now also IC5.1 (INPUT)
- net CH1N_IN renamed CH1_IN_N
- net CH1N_OUT renamed CH1_OUT_N
- net CH1P_IN renamed CH1_IN_P
- net CH1P_OUT renamed CH1_OUT_P
- net CH2N_IN renamed CH2_IN_N
- net CH2N_OUT renamed CH2_OUT_N
- net CH2P_IN renamed CH2_IN_P
- net CH2P_OUT renamed CH2_OUT_P
- new net: C17.1, D5.1 (K), L1.1, U6.2 (OUT)
- new net: C17.2, D5.2 (A)
- new net: L1.2, U6.3 (FB)
- new net: U6.5 (GND), U6.6 (GND), U6.7 (GND), U6.8 (GND)
- new net: C11.1, C12.1, U4.21 (AREF)
- new net: C14.1, U4.9 (XTAL1/PB6), Y1.1
- new net: R14.2, U4.25 (ADC2/PC2)
- new net: D1.2 (A), R18.2
- new net: U5.1 (X1), Y2.1
- new net: U5.2 (X2), Y2.2
- new net: BT1.1 (+), U5.3 (VBAT), VBAT_TP1.1
- new net: C15.1, U4.10 (XTAL2/PB7), Y1.2
- new net: C16.2, J5.6 (Pin_6)
- new net: R13.2, U4.26 (ADC3/PC3)
- new net A4 SDA: U5.5 (SDA)
- new net A5 SCK: U5.6 (SCL)
- new net LCD E: J7.1 (Pin_1)
- new net LOAD MAX: J7.4 (Pin_4)
- new net RXD: J5.5 (Pin_5), RX_TP1.1, U4.2 (RXD/PD0)
- new net SCK: J7.3 (Pin_3), R18.1, U4.19 (SCK/PB5)
- new net TXD: J5.4 (Pin_4), TX_TP1.1, U4.3 (TXD/PD1)
- new net ~{RST}: C16.1, J7.5 (Pin_5), R17.1, SW1.1 (A), SW1.2 (A), U4.1 (~{RESET}/PC6)
- no-connect marks 21 -> 25
Other:
- note added: "6-pos programming header"
- note added: "Aref decoupling"
- note added: "Blinky LED"
- note added: "Crystal Circuit"
- note added: "ICSP"
- note added: "MCU"
- note added: "RTC Module"
- note added: "Reset Button"
- note added: "Reset Logic"
- note added: "Serial"
